Commit message: Imported upstream version '0.0.2' of 'upstream'

File: urdf/coffee_table.urdf.xacro (robot description, xacro)
@@ -23,5 +23,5 @@
     </link>
     <xacro:nav_goal parent="coffee_table" child="coffee_table">
-      <origin xyz="0 -0.6 0" rpy="0 0 0"/>
+      <origin xyz="0 -0.9 0" rpy="0 0 0"/>
     </xacro:nav_goal>
   </xacro:macro>

File: urdf/ilab.urdf.xacro (robot description, xacro)
@@ -30,5 +30,5 @@
   </xacro:kitchen_counter>
   <xacro:kitchen_table parent="${FRAME}">
-    <origin xyz="3.877 5.704 0" rpy="0 0 0" />
+    <origin xyz="3.877 5.66 0" rpy="0 0 ${M_PI/2}" />
   </xacro:kitchen_table>
   <xacro:coffee_table parent="${FRAME}">
@@ -49,8 +49,8 @@
 <!-- THE CHAIRS FACE THE WRONG DIRECTION STILL-->
   <xacro:lazy_chair parent="${FRAME}" suffix="1">
-    <origin xyz="3.64 1.1 0" rpy="0 0 0" />
+    <origin xyz="3.64 1.1 0" rpy="0 0 ${M_PI}" />
   </xacro:lazy_chair>
   <xacro:lazy_chair parent="${FRAME}" suffix="2">
-    <origin xyz="2.621 1.1 0" rpy="0 0 0" />
+    <origin xyz="2.621 1.1 0" rpy="0 0 ${M_PI}" />
   </xacro:lazy_chair>
   <xacro:kitchen_chair parent="${FRAME}">

File: urdf/kitchen_counter.urdf.xacro (robot description, xacro)
@@ -23,5 +23,5 @@
     <link name="sink_link"/>
     <xacro:nav_goal parent="kitchen_counter" child="sink">
-      <origin xyz="0 -0.55 0" rpy="0 0 0"/>
+      <origin xyz="0 -.95 0" rpy="0 0 0"/>
     </xacro:nav_goal>
     <!-- LEFT -->
@@ -34,5 +34,5 @@
     </link>
     <xacro:nav_goal parent="kitchen_counter" child="kitchen_counter_left">
-      <origin xyz="-.6 -0.55 0" rpy="0 0 0"/>
+      <origin xyz="-.6 -.95 0" rpy="0 0 0"/>
     </xacro:nav_goal>
     <!-- RIGHT -->
@@ -45,5 +45,5 @@
     </link>
     <xacro:nav_goal parent="kitchen_counter" child="kitchen_counter_right" >
-      <origin xyz="0.6 -0.55 0" rpy="0 0 0"/>
+      <origin xyz="0.6 -.95 0" rpy="0 0 0"/>
     </xacro:nav_goal>
   </xacro:macro>

File: urdf/kitchen_table.urdf.xacro (robot description, xacro)
@@ -22,5 +22,5 @@
     </link>
     <xacro:nav_goal parent="kitchen_table" child="kitchen_table">
-      <origin xyz="0 -.75 0" rpy="0 0 0"/>
+      <origin xyz="0 -.85 0" rpy="0 0 0"/>
     </xacro:nav_goal>
   </xacro:macro>

File: urdf/left_shelves.urdf.xacro (robot description, xacro)
@@ -15,5 +15,5 @@
     </link>
     <xacro:nav_goal parent="left_shelves" child="left_shelves">
-      <origin xyz="0 -0.52 0" rpy="0 0 0"/>
+      <origin xyz="0 -0.6 0" rpy="0 0 0"/>
     </xacro:nav_goal>
   </xacro:macro>

File: urdf/right_shelves.urdf.xacro (robot description, xacro)
@@ -15,5 +15,5 @@
     </link>
     <xacro:nav_goal parent="right_shelves" child="right_shelves">
-      <origin xyz="0 -0.52 0" rpy="0 0 0"/>
+      <origin xyz="0 -0.6 0" rpy="0 0 0"/>
     </xacro:nav_goal>
   </xacro:macro>

File: urdf/tv.urdf.xacro (robot description, xacro)
@@ -22,5 +22,5 @@
     </link>
     <xacro:nav_goal parent="tv" child="tv">
-      <origin xyz="0 -0.7 0" rpy="0 0 0"/>
+      <origin xyz="0 -0.8 0" rpy="0 0 0"/>
     </xacro:nav_goal>
   </xacro:macro>

Commit message: Imported upstream version '0.0.3' of 'upstream'

File: urdf/coffee_table.urdf.xacro (robot description, xacro)
@@ -15,11 +15,7 @@
       </visual>
     </link>
-    <joint name="${parent}_coffee_table_surface_joint" type="fixed">
-      <origin xyz="0 0 0.41" rpy="0 0 0"/>
-      <parent link="coffee_table_link"/>
-      <child link="coffee_table_surface_link"/>
-    </joint>
-    <link name="coffee_table_surface_link">
-    </link>
+    <xacro:surface parent="coffee_table" child="coffee_table">
+      <origin xyz="0 0 0.5" rpy="0 0 0"/>
+    </xacro:surface>
     <xacro:nav_goal parent="coffee_table" child="coffee_table">
       <origin xyz="0 -0.9 0" rpy="0 0 0"/>

File: urdf/kitchen_table.urdf.xacro (robot description, xacro)
@@ -22,5 +22,5 @@
     </link>
     <xacro:nav_goal parent="kitchen_table" child="kitchen_table">
-      <origin xyz="0 -.85 0" rpy="0 0 0"/>
+      <origin xyz="-1.00 0 0" rpy="0 0 -${M_PI/2}"/>
     </xacro:nav_goal>
   </xacro:macro>

Commit message: Imported upstream version '0.0.4' of 'upstream'

File: urdf/coffee_table.urdf.xacro (robot description, xacro)
@@ -16,8 +16,9 @@
     </link>
     <xacro:surface parent="coffee_table" child="coffee_table">
-      <origin xyz="0 0 0.5" rpy="0 0 0"/>
+      <origin xyz="0 0 0.45" rpy="0 0 0"/>
+      <box size="1.2 0.5 0.05"/>
     </xacro:surface>
     <xacro:nav_goal parent="coffee_table" child="coffee_table">
-      <origin xyz="0 -0.9 0" rpy="0 0 0"/>
+      <origin xyz="0 -0.8 0" rpy="0 0 0"/>
     </xacro:nav_goal>
   </xacro:macro>

File: urdf/ilab.urdf.xacro (robot description, xacro)
@@ -1,4 +1,6 @@
 <?xml version="1.0"?>
 <robot xmlns:xacro="http://www.ros.org/wiki/xacro" name="ilab">
+  <xacro:include filename="$(find rail_collada_models)/urdf/nav_goal.urdf.xacro" />
+  <xacro:include filename="$(find rail_collada_models)/urdf/surface.urdf.xacro" />
   <xacro:include filename="$(find rail_collada_models)/urdf/kitchen_counter.urdf.xacro" />
   <xacro:include filename="$(find rail_collada_models)/urdf/kitchen_chair.urdf.xacro" />
@@ -6,5 +8,4 @@
   <xacro:include filename="$(find rail_collada_models)/urdf/coffee_table.urdf.xacro" />
   <xacro:include filename="$(find rail_collada_models)/urdf/couch.urdf.xacro" />
-  <xacro:include filename="$(find rail_collada_models)/urdf/nav_goal.urdf.xacro" />
   <xacro:include filename="$(find rail_collada_models)/urdf/right_shelves.urdf.xacro" />
   <xacro:include filename="$(find rail_collada_models)/urdf/tv.urdf.xacro" />
@@ -47,5 +48,4 @@
     <origin xyz="0.425 0.838 0" rpy="0 0 ${M_PI/2}" />
   </xacro:left_shelves>
-<!-- THE CHAIRS FACE THE WRONG DIRECTION STILL-->
   <xacro:lazy_chair parent="${FRAME}" suffix="1">
     <origin xyz="3.64 1.1 0" rpy="0 0 ${M_PI}" />

File: urdf/kitchen_counter.urdf.xacro (robot description, xacro)
@@ -26,22 +26,16 @@
     </xacro:nav_goal>
     <!-- LEFT -->
-    <joint name="${parent}_kitchen_counter_left_surface_joint" type="fixed">
+    <xacro:surface parent="kitchen_counter" child="kitchen_counter_left">
       <origin xyz="-0.6 0 0.92" rpy="0 0 0"/>
-      <parent link="kitchen_counter_link" />
-      <child link="kitchen_counter_left_surface_link"/>
-    </joint>
-    <link name="kitchen_counter_left_surface_link">
-    </link>
+      <box size="0.5 0.5 0.05"/>
+    </xacro:surface>
     <xacro:nav_goal parent="kitchen_counter" child="kitchen_counter_left">
       <origin xyz="-.6 -.95 0" rpy="0 0 0"/>
     </xacro:nav_goal>
     <!-- RIGHT -->
-    <joint name="${parent}_kitchen_counter_right_surface_joint" type="fixed">
+    <xacro:surface parent="kitchen_counter" child="kitchen_counter_right">
       <origin xyz="0.6 0 0.92" rpy="0 0 0"/>
-      <parent link="kitchen_counter_link" />
-      <child link="kitchen_counter_right_surface_link"/>
-    </joint>
-    <link name="kitchen_counter_right_surface_link">
-    </link>
+      <box size="0.5 0.5 0.05"/>
+    </xacro:surface>
     <xacro:nav_goal parent="kitchen_counter" child="kitchen_counter_right" >
       <origin xyz="0.6 -.95 0" rpy="0 0 0"/>

File: urdf/kitchen_table.urdf.xacro (robot description, xacro)
@@ -14,11 +14,8 @@
       </visual>
     </link>
-    <joint name="${parent}_kitchen_table_surface_joint" type="fixed">
-      <origin xyz="0 0 0.75" rpy="0 0 0"/>
-      <parent link="kitchen_table_link"/>
-      <child link="kitchen_table_surface_link"/>
-    </joint>
-    <link name="kitchen_table_surface_link">
-    </link>
+    <xacro:surface parent="kitchen_table" child="kitchen_table">
+      <origin xyz="0 0 0.75" rpy="0 0 -${M_PI/2}"/>
+      <box size="0.8 0.8 0.05"/>
+    </xacro:surface>
     <xacro:nav_goal parent="kitchen_table" child="kitchen_table">
       <origin xyz="-1.00 0 0" rpy="0 0 -${M_PI/2}"/>

File: urdf/lazy_chair.urdf.xacro (robot description, xacro)
@@ -5,7 +5,7 @@
       <xacro:insert_block name="origin" />
       <parent link="${parent}" />
-      <child link="lazy_chair_link_${suffix}" />
+      <child link="lazy_chair_${suffix}_link" />
     </joint>
-    <link name="lazy_chair_link_${suffix}">
+    <link name="lazy_chair_${suffix}_link">
       <visual>
         <geometry>
@@ -14,4 +14,8 @@
       </visual>
     </link>
+    <xacro:surface parent="lazy_chair_${suffix}" child="lazy_chair_${suffix}">
+      <origin xyz="0 0 0.48" rpy="0 0 0"/>
+      <box size="0.5 0.5 0.05"/>
+    </xacro:surface>
   </xacro:macro>
 </root>

File: urdf/left_shelves.urdf.xacro (robot description, xacro)
@@ -15,5 +15,5 @@
     </link>
     <xacro:nav_goal parent="left_shelves" child="left_shelves">
-      <origin xyz="0 -0.6 0" rpy="0 0 0"/>
+      <origin xyz="0 -0.7 0" rpy="0 0 0"/>
     </xacro:nav_goal>
   </xacro:macro>

File: urdf/right_shelves.urdf.xacro (robot description, xacro)
@@ -15,5 +15,5 @@
     </link>
     <xacro:nav_goal parent="right_shelves" child="right_shelves">
-      <origin xyz="0 -0.6 0" rpy="0 0 0"/>
+      <origin xyz="0 -0.7 0" rpy="0 0 0"/>
     </xacro:nav_goal>
   </xacro:macro>

File: urdf/surface.urdf.xacro (robot description, xacro)
@@ -1,5 +1,5 @@
 <?xml version="1.0"?>
 <root xmlns:xacro="http://ros.org/wiki/xacro">
-  <xacro:macro name="surface" params="parent child *origin">
+  <xacro:macro name="surface" params="parent child *origin *box">
   	<joint name="${child}_surface_joint" type="fixed">
       <xacro:insert_block name="origin" />
@@ -7,5 +7,11 @@
       <child link="${child}_surface_link"/>
     </joint>
-    <link name="${child}_surface_link"/>
+    <link name="${child}_surface_link">
+    	<collision>
+    		<geometry>
+    			<xacro:insert_block name="box"/>
+    		</geometry>
+    	</collision>
+    </link>
   </xacro:macro>
 </root>

File: urdf/tv.urdf.xacro (robot description, xacro)
@@ -14,11 +14,8 @@
       </visual>
     </link>
-    <joint name="${parent}_tv_surface_joint" type="fixed">
+    <xacro:surface parent="tv" child="tv">
       <origin xyz="0 0 0.605" rpy="0 0 0"/>
-      <parent link="tv_link"/>
-      <child link="tv_surface_link"/>
-    </joint>
-    <link name="tv_surface_link">
-    </link>
+      <box size="0.6 0.35 0.05"/>
+    </xacro:surface>
     <xacro:nav_goal parent="tv" child="tv">
       <origin xyz="0 -0.8 0" rpy="0 0 0"/>
